File: blinds-shield/input-shield/input-shield_for_Adafruit_HUZZAH32_ESP32_Feather.sch (EAGLE design)
At the start: 18 parts

Commit message: Add files via upload
nu shieeeld
Parts:
- removed U$34, U$35: FIDUCIAL_1MM, microbuilder:FIDUCIAL_1MM
- added R_DUMMY_PR1, R_DUMMY_PR2: 0k ohm, rcl:R-EU_0204/7
Connections:
- new net N$4: R5_PR1.2, R_DUMMY_PR1.1
- new net N$5: R6_PR2.2, R_DUMMY_PR2.1
- net N$2: now also R_DUMMY_PR1.2; no longer R5_PR1.2
- net N$3: now also R_DUMMY_PR2.2; no longer R6_PR2.2
Other:
- moved on the sheet: R5_PR1, R6_PR2
Changed lines of the file:
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@@
 <?xml version="1.0" encoding="utf-8"?>
 <!DOCTYPE eagle SYSTEM "eagle.dtd">
-<eagle version="9.3.2">
+<eagle version="9.4.0">
 <drawing>
 <settings>
@@
 <attribute name="YEAR" value=""/>
 </part>
-<part name="U$34" library="microbuilder" deviceset="FIDUCIAL" device="_1MM"/>
-<part name="U$35" library="microbuilder" deviceset="FIDUCIAL" device="_1MM"/>
 <part name="U$31" library="microbuilder" deviceset="MOUNTINGHOLE" device="2.5"/>
 <part name="U$32" library="microbuilder" deviceset="MOUNTINGHOLE" device="2.5"/>
@@
 <part name="GND6" library="supply1" deviceset="GND" device=""/>
 <part name="GND7" library="supply1" deviceset="GND" device=""/>
+<part name="R_DUMMY_PR1" library="rcl" library_urn="urn:adsk.eagle:library:334" deviceset="R-EU_" device="0204/7" package3d_urn="urn:adsk.eagle:package:23498/2" value="0k ohm"/>
+<part name="R_DUMMY_PR2" library="rcl" library_urn="urn:adsk.eagle:library:334" deviceset="R-EU_" device="0204/7" package3d_urn="urn:adsk.eagle:package:23498/2" value="0k ohm"/>
 </parts>
 <sheets>
@@
 <attribute name="YEAR" x="247.0277" y="33.0073" size="1.778" layer="94" ratio="12"/>
 </instance>
-<instance part="U$34" gate="G$1" x="231.14" y="25.4" smashed="yes"/>
-<instance part="U$35" gate="G$1" x="228.6" y="25.4" smashed="yes"/>
 <instance part="U$31" gate="G$1" x="236.22" y="25.4" smashed="yes"/>
 <instance part="U$32" gate="G$1" x="241.3" y="25.4" smashed="yes"/>
@@
 <attribute name="VALUE" x="135.89" y="37.338" size="1.778" layer="96"/>
 </instance>
-<instance part="R6_PR2" gate="G$1" x="96.52" y="88.9" smashed="yes">
-<attribute name="NAME" x="92.71" y="90.3986" size="1.778" layer="95"/>
-<attribute name="VALUE" x="92.71" y="85.598" size="1.778" layer="96"/>
-</instance>
-<instance part="R5_PR1" gate="G$1" x="96.52" y="101.6" smashed="yes">
-<attribute name="NAME" x="92.71" y="103.0986" size="1.778" layer="95"/>
-<attribute name="VALUE" x="92.71" y="98.298" size="1.778" layer="96"/>
+<instance part="R6_PR2" gate="G$1" x="91.44" y="88.9" smashed="yes">
+<attribute name="NAME" x="87.63" y="90.3986" size="1.778" layer="95"/>
+<attribute name="VALUE" x="87.63" y="85.598" size="1.778" layer="96"/>
+</instance>
+<instance part="R5_PR1" gate="G$1" x="91.44" y="101.6" smashed="yes">
+<attribute name="NAME" x="87.63" y="103.0986" size="1.778" layer="95"/>
+<attribute name="VALUE" x="87.63" y="98.298" size="1.778" layer="96"/>
 </instance>
 <instance part="R3_BTN2_PULLDOWN" gate="G$1" x="139.7" y="48.26" smashed="yes">
@@
 <instance part="GND7" gate="1" x="154.94" y="53.34" smashed="yes">
 <attribute name="VALUE" x="152.4" y="50.8" size="1.778" layer="96"/>
+</instance>
+<instance part="R_DUMMY_PR1" gate="G$1" x="101.6" y="101.6" smashed="yes">
+<attribute name="NAME" x="97.79" y="103.0986" size="1.778" layer="95"/>
+<attribute name="VALUE" x="97.79" y="98.298" size="1.778" layer="96"/>
+</instance>
+<instance part="R_DUMMY_PR2" gate="G$1" x="101.6" y="88.9" smashed="yes">
+<attribute name="NAME" x="97.79" y="90.3986" size="1.778" layer="95"/>
+<attribute name="VALUE" x="97.79" y="85.598" size="1.778" layer="96"/>
 </instance>
 </instances>
@@
 <segment>
 <pinref part="R5_PR1" gate="G$1" pin="1"/>
-<wire x1="91.44" y1="101.6" x2="83.82" y2="101.6" width="0.1524" layer="91"/>
 <pinref part="GND2" gate="1" pin="GND"/>
-<wire x1="83.82" y1="101.6" x2="83.82" y2="96.52" width="0.1524" layer="91"/>
+<wire x1="86.36" y1="101.6" x2="83.82" y2="96.52" width="0.1524" layer="91"/>
 </segment>
 <segment>
 <pinref part="R6_PR2" gate="G$1" pin="1"/>
 <pinref part="GND3" gate="1" pin="GND"/>
-<wire x1="91.44" y1="88.9" x2="83.82" y2="88.9" width="0.1524" layer="91"/>
-<wire x1="83.82" y1="88.9" x2="83.82" y2="81.28" width="0.1524" layer="91"/>
+<wire x1="86.36" y1="88.9" x2="83.82" y2="81.28" width="0.1524" layer="91"/>
 </segment>
 <segment>
@@
 <net name="N$2" class="0">
 <segment>
+<pinref part="PR1_(LUMINOSITY)" gate="-2" pin="S"/>
+<pinref part="R_DUMMY_PR1" gate="G$1" pin="2"/>
+</segment>
+</net>
+<net name="N$3" class="0">
+<segment>
+<pinref part="PR2_(LUMINOSITY)" gate="-2" pin="S"/>
+<pinref part="R_DUMMY_PR2" gate="G$1" pin="2"/>
+</segment>
+</net>
+<net name="N$4" class="0">
+<segment>
 <pinref part="R5_PR1" gate="G$1" pin="2"/>
-<pinref part="PR1_(LUMINOSITY)" gate="-2" pin="S"/>
-<wire x1="101.6" y1="101.6" x2="106.68" y2="101.6" width="0.1524" layer="91"/>
-</segment>
-</net>
-<net name="N$3" class="0">
-<segment>
-<pinref part="PR2_(LUMINOSITY)" gate="-2" pin="S"/>
+<pinref part="R_DUMMY_PR1" gate="G$1" pin="1"/>
+</segment>
+</net>
+<net name="N$5" class="0">
+<segment>
 <pinref part="R6_PR2" gate="G$1" pin="2"/>
-<wire x1="106.68" y1="88.9" x2="101.6" y2="88.9" width="0.1524" layer="91"/>
-</segment>
-</net>
+<pinref part="R_DUMMY_PR2" gate="G$1" pin="1"/>
+</segment>
+</net>

Commit message: Add files via upload
A0 and A1 are now connected to photoresistors.
Connections:
- removed net N$2: PR1_(LUMINOSITY)-2.S, R_DUMMY_PR1.2
- removed net N$3: PR2_(LUMINOSITY)-2.S, R_DUMMY_PR2.2
- net 3.3V: now also BTN1_(CLOCKWIZE)-1.S, PR1_(LUMINOSITY)-2.S; no longer BTN1_(CLOCKWIZE)-2.S, PR1_(LUMINOSITY)-1.S
- net A0_DAC2: now also PR1_(LUMINOSITY)-1.S, R_DUMMY_PR1.2
- net A1_DAC1: now also PR2_(LUMINOSITY)-2.S, R_DUMMY_PR2.2
- net IO15_A8: now also BTN1_(CLOCKWIZE)-2.S; no longer BTN1_(CLOCKWIZE)-1.S
Other:
- moved on the sheet: BTN1_(CLOCKWIZE)-1, BTN1_(CLOCKWIZE)-2, PR1_(LUMINOSITY)-1, PR1_(LUMINOSITY)-2
Changed lines of the file:
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@@
 <attribute name="VALUE" x="214.376" y="92.456" size="1.27" layer="96"/>
 </instance>
-<instance part="BTN1_(CLOCKWIZE)" gate="-1" x="114.3" y="63.5" smashed="yes" rot="R180">
+<instance part="BTN1_(CLOCKWIZE)" gate="-1" x="193.04" y="104.14" smashed="yes" rot="R90">
+<attribute name="NAME" x="193.802" y="106.68" size="1.524" layer="95" rot="R90"/>
+<attribute name="VALUE" x="191.643" y="103.378" size="1.778" layer="96" rot="R90"/>
+</instance>
+<instance part="BTN1_(CLOCKWIZE)" gate="-2" x="114.3" y="63.5" smashed="yes" rot="R180">
 <attribute name="NAME" x="101.6" y="64.262" size="1.524" layer="95" rot="R180"/>
 <attribute name="VALUE" x="112.522" y="64.643" size="1.778" layer="96" rot="R180"/>
-</instance>
-<instance part="BTN1_(CLOCKWIZE)" gate="-2" x="193.04" y="104.14" smashed="yes" rot="R90">
-<attribute name="NAME" x="193.802" y="106.68" size="1.524" layer="95" rot="R90"/>
-<attribute name="VALUE" x="191.643" y="103.378" size="1.778" layer="96" rot="R90"/>
 </instance>
 <instance part="BTN2_(AUTOMAGIC)" gate="-1" x="198.12" y="104.14" smashed="yes" rot="R90">
@@
 <attribute name="VALUE" x="57.023" y="95.758" size="1.778" layer="96" rot="R90"/>
 </instance>
-<instance part="PR1_(LUMINOSITY)" gate="-1" x="218.44" y="132.08" smashed="yes" rot="R270">
-<attribute name="NAME" x="217.678" y="129.54" size="1.524" layer="95" rot="R270"/>
-<attribute name="VALUE" x="219.837" y="132.842" size="1.778" layer="96" rot="R270"/>
-</instance>
-<instance part="PR1_(LUMINOSITY)" gate="-2" x="109.22" y="101.6" smashed="yes">
-<attribute name="NAME" x="111.76" y="100.838" size="1.524" layer="95"/>
-<attribute name="VALUE" x="108.458" y="102.997" size="1.778" layer="96"/>
+<instance part="PR1_(LUMINOSITY)" gate="-1" x="114.3" y="101.6" smashed="yes">
+<attribute name="NAME" x="116.84" y="100.838" size="1.524" layer="95"/>
+<attribute name="VALUE" x="113.538" y="102.997" size="1.778" layer="96"/>
+</instance>
+<instance part="PR1_(LUMINOSITY)" gate="-2" x="218.44" y="129.54" smashed="yes" rot="R270">
+<attribute name="NAME" x="217.678" y="127" size="1.524" layer="95" rot="R270"/>
+<attribute name="VALUE" x="219.837" y="130.302" size="1.778" layer="96" rot="R270"/>
 </instance>
 <instance part="PR2_(LUMINOSITY)" gate="-1" x="233.68" y="132.08" smashed="yes" rot="R270">
@@
 <wire x1="203.2" y1="83.82" x2="198.12" y2="83.82" width="0.1524" layer="91"/>
 <junction x="203.2" y="83.82"/>
-<wire x1="198.12" y1="83.82" x2="193.04" y2="83.82" width="0.1524" layer="91"/>
 <pinref part="BTN2_(AUTOMAGIC)" gate="-1" pin="S"/>
 <wire x1="198.12" y1="101.6" x2="198.12" y2="83.82" width="0.1524" layer="91"/>
+<wire x1="198.12" y1="83.82" x2="193.04" y2="83.82" width="0.1524" layer="91"/>
 <junction x="198.12" y="83.82"/>
-<pinref part="BTN1_(CLOCKWIZE)" gate="-2" pin="S"/>
-<wire x1="193.04" y1="101.6" x2="193.04" y2="83.82" width="0.1524" layer="91"/>
+<pinref part="BTN1_(CLOCKWIZE)" gate="-1" pin="S"/>
+<wire x1="193.04" y1="83.82" x2="193.04" y2="101.6" width="0.1524" layer="91"/>
 </segment>
 <segment>
@@
 <wire x1="226.06" y1="144.78" x2="226.06" y2="139.7" width="0.1524" layer="91"/>
 <wire x1="226.06" y1="139.7" x2="218.44" y2="139.7" width="0.1524" layer="91"/>
-<wire x1="218.44" y1="139.7" x2="218.44" y2="134.62" width="0.1524" layer="91"/>
 <wire x1="226.06" y1="139.7" x2="233.68" y2="139.7" width="0.1524" layer="91"/>
 <wire x1="233.68" y1="139.7" x2="233.68" y2="134.62" width="0.1524" layer="91"/>
 <junction x="226.06" y="139.7"/>
 <pinref part="PR2_(LUMINOSITY)" gate="-1" pin="S"/>
-<pinref part="PR1_(LUMINOSITY)" gate="-1" pin="S"/>
+<pinref part="PR1_(LUMINOSITY)" gate="-2" pin="S"/>
+<wire x1="218.44" y1="139.7" x2="218.44" y2="132.08" width="0.1524" layer="91"/>
 </segment>
 </net>
@@
 <segment>
 <pinref part="JP1" gate="A" pin="11"/>
-<wire x1="236.22" y1="73.66" x2="215.9" y2="73.66" width="0.1524" layer="91"/>
 <label x="215.9" y="73.66" size="1.778" layer="95"/>
+<wire x1="236.22" y1="73.66" x2="187.96" y2="73.66" width="0.1524" layer="91"/>
+<wire x1="187.96" y1="73.66" x2="187.96" y2="93.98" width="0.1524" layer="91"/>
+<wire x1="187.96" y1="93.98" x2="106.68" y2="93.98" width="0.1524" layer="91"/>
+<pinref part="PR2_(LUMINOSITY)" gate="-2" pin="S"/>
+<pinref part="R_DUMMY_PR2" gate="G$1" pin="2"/>
+<wire x1="106.68" y1="93.98" x2="106.68" y2="88.9" width="0.1524" layer="91"/>
+<junction x="106.68" y="88.9"/>
 </segment>
 </net>
 <net name="A0_DAC2" class="0">
 <segment>
-<wire x1="236.22" y1="76.2" x2="215.9" y2="76.2" width="0.1524" layer="91"/>
 <pinref part="JP1" gate="A" pin="12"/>
 <label x="215.9" y="76.2" size="1.778" layer="95"/>
+<wire x1="236.22" y1="76.2" x2="190.5" y2="76.2" width="0.1524" layer="91"/>
+<wire x1="190.5" y1="76.2" x2="190.5" y2="101.6" width="0.1524" layer="91"/>
+<wire x1="190.5" y1="101.6" x2="149.86" y2="101.6" width="0.1524" layer="91"/>
+<wire x1="149.86" y1="101.6" x2="149.86" y2="109.22" width="0.1524" layer="91"/>
+<wire x1="149.86" y1="109.22" x2="109.22" y2="109.22" width="0.1524" layer="91"/>
+<pinref part="PR1_(LUMINOSITY)" gate="-1" pin="S"/>
+<pinref part="R_DUMMY_PR1" gate="G$1" pin="2"/>
+<wire x1="111.76" y1="101.6" x2="109.22" y2="101.6" width="0.1524" layer="91"/>
+<wire x1="109.22" y1="101.6" x2="106.68" y2="101.6" width="0.1524" layer="91"/>
+<wire x1="109.22" y1="109.22" x2="109.22" y2="101.6" width="0.1524" layer="91"/>
+<junction x="109.22" y="101.6"/>
 </segment>
 </net>
@@
 <label x="160.02" y="63.5" size="1.778" layer="95"/>
 <pinref part="JP3" gate="G$1" pin="8"/>
-<pinref part="BTN1_(CLOCKWIZE)" gate="-1" pin="S"/>
-<wire x1="127" y1="63.5" x2="116.84" y2="63.5" width="0.1524" layer="91"/>
 <wire x1="127" y1="63.5" x2="127" y2="48.26" width="0.1524" layer="91"/>
-<junction x="127" y="63.5"/>
 <pinref part="R3_BTN2_PULLDOWN" gate="G$1" pin="1"/>
 <wire x1="127" y1="48.26" x2="134.62" y2="48.26" width="0.1524" layer="91"/>
+<pinref part="BTN1_(CLOCKWIZE)" gate="-2" pin="S"/>
+<wire x1="116.84" y1="63.5" x2="127" y2="63.5" width="0.1524" layer="91"/>
+<junction x="127" y="63.5"/>
 </segment>
 </net>
@@
 </segment>
 </net>
-<net name="N$2" class="0">
-<segment>
-<pinref part="PR1_(LUMINOSITY)" gate="-2" pin="S"/>
-<pinref part="R_DUMMY_PR1" gate="G$1" pin="2"/>
-</segment>
-</net>
-<net name="N$3" class="0">
-<segment>
-<pinref part="PR2_(LUMINOSITY)" gate="-2" pin="S"/>
-<pinref part="R_DUMMY_PR2" gate="G$1" pin="2"/>
-</segment>
-</net>
